Commit message: Adjusted controls b/c some controls just make robot take flight - :) - also removing more comments from xacro

File: hyperdog_gazebo_sim/description/hyperdog_urdf_links.xacro (robot description, xacro)
@@ -259,24 +259,24 @@
     <link name="FL_foot">
         <visual>
-          <origin rpy="0 0 0" xyz="0 0 0"/>
-          <geometry>
-            <sphere radius="${foot_radius}"/>
-          </geometry>
-          <material name="orange"/>
-        </visual>
-        <collision>
-          <origin rpy="0 0 0" xyz="0 0 0"/>
-          <geometry>
-            <sphere radius="${foot_radius}"/>
-          </geometry>
-          <surface>
-            <friction>
-                <ode>
-                    <mu>1</mu>
-                    <mu2>1</mu2>
-                    <fdir1>1 0 0</fdir1>
-                </ode>
-            </friction>
-        </surface>
+            <origin rpy="0 0 0" xyz="0 0 0"/>
+            <geometry>
+                <sphere radius="${foot_radius}"/>
+            </geometry>
+            <material name="orange"/>
+        </visual>
+        <collision>
+            <origin rpy="0 0 0" xyz="0 0 0"/>
+            <geometry>
+                <sphere radius="${foot_radius}"/>
+            </geometry>
+            <surface>
+                <friction>
+                    <ode>
+                        <mu>1</mu>
+                        <mu2>1</mu2>
+                        <fdir1>1 0 0</fdir1>
+                    </ode>
+                </friction>
+            </surface>
         </collision>
         <xacro:inertial_foot></xacro:inertial_foot>
@@ -284,24 +284,24 @@
     <link name="FR_foot">
         <visual>
-          <origin rpy="0 0 0" xyz="0 0 0"/>
-          <geometry>
-            <sphere radius="${foot_radius}"/>
-          </geometry>
-          <material name="orange"/>
-        </visual>
-        <collision>
-          <origin rpy="0 0 0" xyz="0 0 0"/>
-          <geometry>
-            <sphere radius="${foot_radius}"/>
-          </geometry>
-          <surface>
-            <friction>
-                <ode>
-                    <mu>1</mu>
-                    <mu2>1</mu2>
-                    <fdir1>1 0 0</fdir1>
-                </ode>
-            </friction>
-        </surface>
+            <origin rpy="0 0 0" xyz="0 0 0"/>
+            <geometry>
+                <sphere radius="${foot_radius}"/>
+            </geometry>
+            <material name="orange"/>
+        </visual>
+        <collision>
+            <origin rpy="0 0 0" xyz="0 0 0"/>
+            <geometry>
+                <sphere radius="${foot_radius}"/>
+            </geometry>
+            <surface>
+                <friction>
+                    <ode>
+                        <mu>1</mu>
+                        <mu2>1</mu2>
+                        <fdir1>1 0 0</fdir1>
+                    </ode>
+                </friction>
+            </surface>
         </collision>
         <xacro:inertial_foot></xacro:inertial_foot>
@@ -309,24 +309,24 @@
     <link name="BR_foot">
         <visual>
-          <origin rpy="0 0 0" xyz="0 0 0"/>
-          <geometry>
-            <sphere radius="${foot_radius}"/>
-          </geometry>
-          <material name="orange"/>
-        </visual>
-        <collision>
-          <origin rpy="0 0 0" xyz="0 0 0"/>
-          <geometry>
-            <sphere radius="${foot_radius}"/>
-          </geometry>
-          <surface>
-            <friction>
-                <ode>
-                    <mu>1</mu>
-                    <mu2>1</mu2>
-                    <fdir1>1 0 0</fdir1>
-                </ode>
-            </friction>
-        </surface>
+            <origin rpy="0 0 0" xyz="0 0 0"/>
+            <geometry>
+                <sphere radius="${foot_radius}"/>
+            </geometry>
+            <material name="orange"/>
+        </visual>
+        <collision>
+            <origin rpy="0 0 0" xyz="0 0 0"/>
+            <geometry>
+                <sphere radius="${foot_radius}"/>
+            </geometry>
+            <surface>
+                <friction>
+                    <ode>
+                        <mu>1</mu>
+                        <mu2>1</mu2>
+                        <fdir1>1 0 0</fdir1>
+                    </ode>
+                </friction>
+            </surface>
         </collision>
         <xacro:inertial_foot></xacro:inertial_foot>
@@ -334,24 +334,24 @@
     <link name="BL_foot">
         <visual>
-          <origin rpy="0 0 0" xyz="0.0 0 0"/>
-          <geometry>
-            <sphere radius="${foot_radius}"/>
-          </geometry>
-          <material name="orange"/>
-        </visual>
-        <collision>
-          <origin rpy="0 0 0" xyz="0 0 0"/>
-          <geometry>
-            <sphere radius="${foot_radius}"/>
-          </geometry>
-          <surface>
-            <friction>
-                <ode>
-                    <mu>1</mu>
-                    <mu2>1</mu2>
-                    <fdir1>1 0 0</fdir1>
-                </ode>
-            </friction>
-        </surface>
+            <origin rpy="0 0 0" xyz="0 0 0"/>
+            <geometry>
+                <sphere radius="${foot_radius}"/>
+            </geometry>
+            <material name="orange"/>
+        </visual>
+        <collision>
+            <origin rpy="0 0 0" xyz="0 0 0"/>
+            <geometry>
+                <sphere radius="${foot_radius}"/>
+            </geometry>
+            <surface>
+                <friction>
+                    <ode>
+                        <mu>1</mu>
+                        <mu2>1</mu2>
+                        <fdir1>1 0 0</fdir1>
+                    </ode>
+                </friction>
+            </surface>
         </collision>
         <xacro:inertial_foot></xacro:inertial_foot>

File: hyperdog_gazebo_sim/description/physics.xacro (robot description, xacro)
@@ -2,13 +2,11 @@
 <robot xmlns:xacro="http://www.ros.org/wiki/xacro" >
     <xacro:include filename="consts.xacro" />
-    <!--  BODY -->
     <xacro:macro name="inertial_body">
         <inertial>
-            <origin xyz="-0.006 0.00633 0.00214" rpy="0 0 0"/> <!-- 0.006, -0.000233, 0.00214 -->
+            <origin xyz="-0.006 0.00633 0.00214" rpy="0 0 0"/>
             <mass value="${body_mass}" />
             <inertia  ixx="0.011396658109874464" ixy="0" ixz="0" iyy="0.05486450023370329" iyz="0" izz="0.06098759357764758" />
         </inertial>
     </xacro:macro>
-    <!-- HIP -->
     <xacro:macro name="inertial_right_hip">
         <inertial>
@@ -25,5 +23,4 @@
         </inertial>
     </xacro:macro>
-    <!-- ULEG -->
     <xacro:macro name="inertial_right_uleg">
         <inertial>
@@ -40,5 +37,4 @@
         </inertial>
     </xacro:macro>
-    <!-- LLEG -->
     <xacro:macro name="inertial_right_lleg">
         <inertial>
@@ -55,5 +51,4 @@
         </inertial>
     </xacro:macro>
-    <!-- FOOT -->
     <xacro:macro name="inertial_foot">
         <inertial>
@@ -65,4 +60,3 @@
         </inertial>
     </xacro:macro>
-    <!-- ************************************************************************************************** -->
 </robot>
